File: uno-r4-shield-template.kicad_pcb (KiCad board)
At the start: 2 copper layers, 150.8 x 112.1 mm, 88 parts, among them J1 POWER1, J10 +5V output, J11 +3.3V output, J12 Solder Pads 2, J13 GND, J14 Pin17 Rasp Pi LED Green, J15 Pilot Lamp Buzzer, J16 220VAC Detection In, J17 220VAC Detection Out, J19 GSM LED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

Commit message: Add files via upload
Parts:
- removed D5: LED, LED_THT:LED_D3.0mm
- removed J10: +5V output, TerminalBlock_Phoenix:TerminalBlock_Phoenix_MKDS-1,5-2-5.08_1x02_P5.08mm_Horizontal
- removed J11: +3.3V output, TerminalBlock_Phoenix:TerminalBlock_Phoenix_MKDS-1,5-2-5.08_1x02_P5.08mm_Horizontal
- removed R10: 10KΩ, Resistor_THT:R_Axial_DIN0207_L6.3mm_D2.5mm_P10.16mm_Horizontal
- removed U4: EL817, Package_DIP:DIP-4_W7.62mm
- added J18: GSM LED, Connector_PinHeader_2.54mm:PinHeader_1x02_P2.54mm_Vertical, F.Cu at (205.0, 99.4)
- added Q4: BSS138, Package_TO_SOT_SMD:SOT-23, F.Cu at (183.7, 65.1)
- added R3: 10k, +-5%, Resistor_THT:R_Axial_DIN0204_L3.6mm_D1.6mm_P5.08mm_Horizontal, F.Cu at (193.8, 64.4)
- J19: value GSM LED -> Buzzer Enable; footprint Connector_PinHeader_2.54mm:PinHeader_1x01_P2.54mm_Vertical -> Connector_PinHeader_2.54mm:PinHeader_1x02_P2.54mm_Vertical
- J3: value GSM Orange LED -> GSM LED Orange
- R8: value 510Ω -> 10k, +-5%; footprint Resistor_THT:R_Axial_DIN0207_L6.3mm_D2.5mm_P10.16mm_Horizontal -> Resistor_THT:R_Axial_DIN0204_L3.6mm_D1.6mm_P5.08mm_Horizontal
- moved R8 74.9 mm to (194.6, 67.5), turned to 0 degrees
- moved J19 38.9 mm to (200.2, 140.8), turned to -90 degrees
- moved Q3 11.7 mm to (169.9, 118.9)
- moved R9 11.7 mm to (171.2, 122.6)
- moved D6 11.7 mm to (186.2, 119.1)
- moved K3 11.7 mm to (174.8, 135.6)
- moved J15 11.7 mm to (206.5, 135.5)
Connections:
- GSM_Module1 pad 5: D3~ -> GSM_TXD
- J15 pad 1: Pilot_Lamp -> Pilot_Lamp_Out
- J17 pad 1: GND -> Net-(J17-Pin_1)
- J17 pad 2: Net-(J17-Pin_2) -> unconnected-(J17-Pin_2-Pad2)
- J19 pad 1: Net-(J19-Pin_1) -> Pilot_Lamp_Out
- J3 pad 1: Net-(J19-Pin_1) -> Net-(J18-Pin_1)
- K3 pad 3: Pilot_Lamp -> unconnected-(K3-Pad3)
- K3 pad 4: unconnected-(K3-Pad4) -> Pilot_Lamp
- R8 pad 1: Net-(R8-Pad1) -> GSM_TXD
- R8 pad 2: Net-(J17-Pin_2) -> +3.3V
- R9 pad 2: Net-(R9-Pad2) -> Net-(J17-Pin_1)
Routing:
- net Net-(J19-Pin_1): track 61.8 -> 0.00 mm
- net Net-(J18-Pin_1): track 0.00 -> 61.8 mm
- net Net-(J17-Pin_1): track 0.00 -> 39.3 mm
- net +3.3V: track 311.7 -> 282.6 mm
- net +5V: track 54.8 -> 79.0 mm, vias 0 -> 2
- net GND: track 25.8 -> 2.97 mm
- net Net-(J17-Pin_2): track 19.9 -> 0.00 mm
- net GSM_TXD: track 0.00 -> 19.6 mm
- net +12V: track 227.2 -> 217.4 mm
- net Pilot_Lamp_Out: track 0.00 -> 9.52 mm
- net D3~: track 23.8 -> 18.6 mm
- net Pilot_Lamp: track 15.1 -> 19.7 mm
- net Net-(D5-A): track 4.17 -> 0.00 mm
- net Net-(R8-Pad1): track 3.98 -> 0.00 mm
- net Net-(R9-Pad2): track 3.02 -> 0.00 mm
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Other:
- board size 150.8 x 112.1 mm -> 137.8 x 112.1 mm
- board text added: "Pin17 Coin En"
- board text added: "Pin27 LED"
- board text added: "SIM800L Arduino Shield By DJ Tar v2.1"
- board text removed: "+3.3V"
- board text removed: "+5V"
- board text removed: "Pin17 LED"
- board text removed: "Pin27 Coin En"
- board text removed: "SIM800L Arduino Shield By DJ Tar v2.0"
